File: rev1.a/SmartiePiNode.sch (KiCad schematic (older format))
At the start: 48 parts, among them CN1 USBMICROb, CN2 ST-LINK, CN3 SX1238_TRX_HEADER, SW1 SW_PUSH, U1 ISL91127IR, U2 STM32L052_LQFP48, X2 ABS25-32.768KHZ-6-T

Commit message: starting pcb layout/design
Parts:
- added H1, H2, H3, H4: m3-mounting-hole, m3-mounting-holes:m3-mounting-hole, symbol m3-mounting-hole
- CN3: footprint Pin_Headers:Pin_Header_Straight_2x10 -> Socket_Strips:Socket_Strip_Straight_2x10
- X1: renamed from X?; footprint (none) -> abracon-abm10:abracon-abm10
Connections:
- net GND: now also H1.1, H2.1, H3.1, H4.1
Changed lines of the file:
@@
 LIBS:crystal_small
 LIBS:abracon-abm10
+LIBS:m3-mounting-hole
 LIBS:SmartiePiNode-cache
 EELAYER 26 0
@@
 $EndComp
 $Comp
-L GND #PWR01
+L GND #PWR10
 U 1 1 5B041A53
 P 3720 7315
-F 0 "#PWR01" H 3720 7065 50  0001 C CNN
+F 0 "#PWR10" H 3720 7065 50  0001 C CNN
 F 1 "GND" H 3725 7142 50  0000 C CNN
 F 2 "" H 3720 7315 50  0001 C CNN
@@
 $EndComp
 $Comp
-L GND #PWR02
+L GND #PWR15
 U 1 1 5B041F18
 P 4975 6485
-F 0 "#PWR02" H 4975 6235 50  0001 C CNN
+F 0 "#PWR15" H 4975 6235 50  0001 C CNN
 F 1 "GND" H 4980 6312 50  0000 C CNN
 F 2 "" H 4975 6485 50  0001 C CNN
@@
 $EndComp
 $Comp
-L GND #PWR03
+L GND #PWR16
 U 1 1 5B04234F
 P 5255 6485
-F 0 "#PWR03" H 5255 6235 50  0001 C CNN
+F 0 "#PWR16" H 5255 6235 50  0001 C CNN
 F 1 "GND" H 5260 6312 50  0000 C CNN
 F 2 "" H 5255 6485 50  0001 C CNN
@@
 $EndComp
 $Comp
-L GND #PWR04
+L GND #PWR17
 U 1 1 5B0423C8
 P 5530 6485
-F 0 "#PWR04" H 5530 6235 50  0001 C CNN
+F 0 "#PWR17" H 5530 6235 50  0001 C CNN
 F 1 "GND" H 5535 6312 50  0000 C CNN
 F 2 "" H 5530 6485 50  0001 C CNN
@@
 $EndComp
 $Comp
-L GND #PWR05
+L GND #PWR6
 U 1 1 5B04306E
 P 2340 6485
-F 0 "#PWR05" H 2340 6235 50  0001 C CNN
+F 0 "#PWR6" H 2340 6235 50  0001 C CNN
 F 1 "GND" H 2345 6312 50  0000 C CNN
 F 2 "" H 2340 6485 50  0001 C CNN
@@
 $EndComp
 $Comp
-L GND #PWR06
+L GND #PWR4
 U 1 1 5B04307C
 P 2060 6485
-F 0 "#PWR06" H 2060 6235 50  0001 C CNN
+F 0 "#PWR4" H 2060 6235 50  0001 C CNN
 F 1 "GND" H 2065 6312 50  0000 C CNN
 F 2 "" H 2060 6485 50  0001 C CNN
@@
 $EndComp
 $Comp
-L GND #PWR07
+L GND #PWR3
 U 1 1 5B04308A
 P 1785 6485
-F 0 "#PWR07" H 1785 6235 50  0001 C CNN
+F 0 "#PWR3" H 1785 6235 50  0001 C CNN
 F 1 "GND" H 1790 6312 50  0000 C CNN
 F 2 "" H 1785 6485 50  0001 C CNN
@@
 $EndComp
 $Comp
-L GND #PWR08
+L GND #PWR7
 U 1 1 5B043F5D
 P 2705 7280
-F 0 "#PWR08" H 2705 7030 50  0001 C CNN
+F 0 "#PWR7" H 2705 7030 50  0001 C CNN
 F 1 "GND" H 2710 7107 50  0000 C CNN
 F 2 "" H 2705 7280 50  0001 C CNN
@@
 $EndComp
 $Comp
-L GND #PWR09
+L GND #PWR12
 U 1 1 5B044D4C
 P 4485 7315
-F 0 "#PWR09" H 4485 7065 50  0001 C CNN
+F 0 "#PWR12" H 4485 7065 50  0001 C CNN
 F 1 "GND" H 4490 7142 50  0000 C CNN
 F 2 "" H 4485 7315 50  0001 C CNN
@@
 $EndComp
 $Comp
-L GND #PWR010
+L GND #PWR22
 U 1 1 5B06F6EF
 P 9930 3790
-F 0 "#PWR010" H 9930 3540 50  0001 C CNN
+F 0 "#PWR22" H 9930 3540 50  0001 C CNN
 F 1 "GND" H 9935 3617 50  0000 C CNN
 F 2 "" H 9930 3790 50  0001 C CNN
@@
 $EndComp
 $Comp
-L GND #PWR011
+L GND #PWR20
 U 1 1 5B0753BB
 P 6760 3380
-F 0 "#PWR011" H 6760 3130 50  0001 C CNN
+F 0 "#PWR20" H 6760 3130 50  0001 C CNN
 F 1 "GND" H 6765 3207 50  0000 C CNN
 F 2 "" H 6760 3380 50  0001 C CNN
@@
 NoConn ~ 1465 4560
 $Comp
-L GND #PWR012
+L GND #PWR1
 U 1 1 5B081C3A
 P 1545 4710
-F 0 "#PWR012" H 1545 4460 50  0001 C CNN
+F 0 "#PWR1" H 1545 4460 50  0001 C CNN
 F 1 "GND" H 1550 4537 50  0000 C CNN
 F 2 "" H 1545 4710 50  0001 C CNN
@@
 $EndComp
 $Comp
-L GND #PWR013
+L GND #PWR18
 U 1 1 5B082DC4
 P 5880 3240
-F 0 "#PWR013" H 5880 2990 50  0001 C CNN
+F 0 "#PWR18" H 5880 2990 50  0001 C CNN
 F 1 "GND" H 5885 3067 50  0000 C CNN
 F 2 "" H 5880 3240 50  0001 C CNN
@@
 Connection ~ 10575 2935
 $Comp
-L GND #PWR015
+L GND #PWR23
 U 1 1 5B098D9A
 P 11070 2830
-F 0 "#PWR015" H 11070 2580 50  0001 C CNN
+F 0 "#PWR23" H 11070 2580 50  0001 C CNN
 F 1 "GND" H 11075 2657 50  0000 C CNN
 F 2 "" H 11070 2830 50  0001 C CNN
@@
 F 0 "CN3" H 3835 1100 50  0000 C CNN
 F 1 "SX1238_TRX_HEADER" H 3895 2224 50  0000 C CNN
-F 2 "Pin_Headers:Pin_Header_Straight_2x10" H 3895 450 50  0001 C CNN
+F 2 "Socket_Strips:Socket_Strip_Straight_2x10" H 3895 450 50  0001 C CNN
 F 3 "" H 3895 450 50  0001 C CNN
 	1    3895 1650
@@
 	2225 1540 2225 1670
 $Comp
-L GND #PWR016
+L GND #PWR5
 U 1 1 5B0A5E1E
 P 2225 1670
-F 0 "#PWR016" H 2225 1420 50  0001 C CNN
+F 0 "#PWR5" H 2225 1420 50  0001 C CNN
 F 1 "GND" H 2230 1497 50  0000 C CNN
 F 2 "" H 2225 1670 50  0001 C CNN
@@
 +3V3
 $Comp
-L GND #PWR017
+L GND #PWR8
 U 1 1 5B0AC996
 P 3070 1200
-F 0 "#PWR017" H 3070 950 50  0001 C CNN
+F 0 "#PWR8" H 3070 950 50  0001 C CNN
 F 1 "GND" H 3075 1027 50  0000 C CNN
 F 2 "" H 3070 1200 50  0001 C CNN
@@
 SPI2_SCK
 $Comp
-L GND #PWR018
+L GND #PWR9
 U 1 1 5B0AE690
 P 3070 1500
-F 0 "#PWR018" H 3070 1250 50  0001 C CNN
+F 0 "#PWR9" H 3070 1250 50  0001 C CNN
 F 1 "GND" H 3075 1327 50  0000 C CNN
 F 2 "" H 3070 1500 50  0001 C CNN
@@
 	4145 2100 4720 2100
 $Comp
-L GND #PWR019
+L GND #PWR13
 U 1 1 5B0AEB87
 P 4720 2100
-F 0 "#PWR019" H 4720 1850 50  0001 C CNN
+F 0 "#PWR13" H 4720 1850 50  0001 C CNN
 F 1 "GND" H 4725 1927 50  0000 C CNN
 F 2 "" H 4720 2100 50  0001 C CNN
@@
 	1625 3160 1695 3160
 $Comp
-L GND #PWR020
+L GND #PWR2
 U 1 1 5B0B10C1
 P 1695 3160
-F 0 "#PWR020" H 1695 2910 50  0001 C CNN
+F 0 "#PWR2" H 1695 2910 50  0001 C CNN
 F 1 "GND" H 1700 2987 50  0000 C CNN
 F 2 "" H 1695 3160 50  0001 C CNN
@@
 NRST
 $Comp
-L GND #PWR021
+L GND #PWR11
 U 1 1 5B0B8F14
 P 4200 3080
-F 0 "#PWR021" H 4200 2830 50  0001 C CNN
+F 0 "#PWR11" H 4200 2830 50  0001 C CNN
 F 1 "GND" H 4205 2907 50  0000 C CNN
 F 2 "" H 4200 3080 50  0001 C CNN
@@
 $EndComp
 $Comp
-L GND #PWR022
+L GND #PWR21
 U 1 1 5B0C38AE
 P 8160 5860
-F 0 "#PWR022" H 8160 5610 50  0001 C CNN
+F 0 "#PWR21" H 8160 5610 50  0001 C CNN
 F 1 "GND" H 8165 5687 50  0000 C CNN
 F 2 "" H 8160 5860 50  0001 C CNN
@@
 $EndComp
 $Comp
-L abracon-abm10 X?
+L abracon-abm10 X1
 U 1 1 5B1A86B5
 P 6260 2395
-F 0 "X?" H 6410 2325 60  0000 C CNN
+F 0 "X1" H 6410 2325 60  0000 C CNN
 F 1 "abm10" H 6265 2565 60  0000 C CNN
-F 2 "" H 6260 2395 60  0001 C CNN
+F 2 "abracon-abm10:abracon-abm10" H 6260 2395 60  0001 C CNN
 F 3 "" H 6260 2395 60  0001 C CNN
 	1    6260 2395
@@
 Connection ~ 6235 2750
 $Comp
-L GND #PWR?
+L GND #PWR19
 U 1 1 5B1AE42D
 P 6235 2785
-F 0 "#PWR?" H 6235 2535 50  0001 C CNN
+F 0 "#PWR19" H 6235 2535 50  0001 C CNN
 F 1 "GND" H 6315 2770 50  0000 C CNN
 F 2 "" H 6235 2785 50  0001 C CNN
@@
 	1    0    0    -1
 $EndComp
+$Comp
+L m3-mounting-hole H1
+U 1 1 5B1D3AA5
+P 5175 4565
+F 0 "H1" H 5110 4480 60  0000 L CNN
+F 1 "m3-mounting-hole" H 5253 4517 60  0000 L CNN
+F 2 "m3-mounting-holes:m3-mounting-hole" H 5175 4565 60  0001 C CNN
+F 3 "" H 5175 4565 60  0001 C CNN
+	1    5175 4565
+	1    0    0    -1
+$EndComp
+$Comp
+L m3-mounting-hole H2
+U 1 1 5B1D3C74
+P 5175 4740
+F 0 "H2" H 5110 4655 60  0000 L CNN
+F 1 "m3-mounting-hole" H 5220 4745 60  0000 L CNN
+F 2 "m3-mounting-holes:m3-mounting-hole" H 5175 4740 60  0001 C CNN
+F 3 "" H 5175 4740 60  0001 C CNN
+	1    5175 4740
+	1    0    0    -1
+$EndComp
+$Comp
+L m3-mounting-hole H3
+U 1 1 5B1D4190
+P 5175 4915
+F 0 "H3" H 5110 4830 60  0000 L CNN
+F 1 "m3-mounting-hole" H 5220 4920 60  0000 L CNN
+F 2 "m3-mounting-holes:m3-mounting-hole" H 5175 4915 60  0001 C CNN
+F 3 "" H 5175 4915 60  0001 C CNN
+	1    5175 4915
+	1    0    0    -1
+$EndComp
+$Comp
+L m3-mounting-hole H4
+U 1 1 5B1D42C3
+P 5175 5090
+F 0 "H4" H 5110 5005 60  0000 L CNN
+F 1 "m3-mounting-hole" H 5220 5095 60  0000 L CNN
+F 2 "m3-mounting-holes:m3-mounting-hole" H 5175 5090 60  0001 C CNN
+F 3 "" H 5175 5090 60  0001 C CNN
+	1    5175 5090
+	1    0    0    -1
+$EndComp
+Wire Wire Line
+	5025 4565 4855 4565
+Wire Wire Line
+	4855 4565 4855 5170
+$Comp
+L GND #PWR14
+U 1 1 5B1D46F6
+P 4855 5170
+F 0 "#PWR14" H 4855 4920 50  0001 C CNN
+F 1 "GND" H 4860 4997 50  0000 C CNN
+F 2 "" H 4855 5170 50  0001 C CNN
+F 3 "" H 4855 5170 50  0001 C CNN
+	1    4855 5170
+	1    0    0    -1
+$EndComp
+Wire Wire Line
+	5025 4740 4855 4740
+Connection ~ 4855 4740
+Wire Wire Line
+	5025 4915 4855 4915
+Connection ~ 4855 4915
+Wire Wire Line
+	5025 5090 4855 5090
+Connection ~ 4855 5090
 $EndSCHEMATC

Commit message: footprint for sx1238 trx module
Parts:
- CN3: footprint Socket_Strips:Socket_Strip_Straight_2x10 -> socket-strip-straight-2x10:sx1238_trx
Changed lines of the file:
@@
 $EndComp
 $Comp
-L GND #PWR10
+L GND #PWR01
 U 1 1 5B041A53
 P 3720 7315
-F 0 "#PWR10" H 3720 7065 50  0001 C CNN
+F 0 "#PWR01" H 3720 7065 50  0001 C CNN
 F 1 "GND" H 3725 7142 50  0000 C CNN
 F 2 "" H 3720 7315 50  0001 C CNN
@@
 $EndComp
 $Comp
-L GND #PWR15
+L GND #PWR02
 U 1 1 5B041F18
 P 4975 6485
-F 0 "#PWR15" H 4975 6235 50  0001 C CNN
+F 0 "#PWR02" H 4975 6235 50  0001 C CNN
 F 1 "GND" H 4980 6312 50  0000 C CNN
 F 2 "" H 4975 6485 50  0001 C CNN
@@
 $EndComp
 $Comp
-L GND #PWR16
+L GND #PWR03
 U 1 1 5B04234F
 P 5255 6485
-F 0 "#PWR16" H 5255 6235 50  0001 C CNN
+F 0 "#PWR03" H 5255 6235 50  0001 C CNN
 F 1 "GND" H 5260 6312 50  0000 C CNN
 F 2 "" H 5255 6485 50  0001 C CNN
@@
 $EndComp
 $Comp
-L GND #PWR17
+L GND #PWR04
 U 1 1 5B0423C8
 P 5530 6485
-F 0 "#PWR17" H 5530 6235 50  0001 C CNN
+F 0 "#PWR04" H 5530 6235 50  0001 C CNN
 F 1 "GND" H 5535 6312 50  0000 C CNN
 F 2 "" H 5530 6485 50  0001 C CNN
@@
 $EndComp
 $Comp
-L GND #PWR6
+L GND #PWR05
 U 1 1 5B04306E
 P 2340 6485
-F 0 "#PWR6" H 2340 6235 50  0001 C CNN
+F 0 "#PWR05" H 2340 6235 50  0001 C CNN
 F 1 "GND" H 2345 6312 50  0000 C CNN
 F 2 "" H 2340 6485 50  0001 C CNN
@@
 $EndComp
 $Comp
-L GND #PWR4
+L GND #PWR06
 U 1 1 5B04307C
 P 2060 6485
-F 0 "#PWR4" H 2060 6235 50  0001 C CNN
+F 0 "#PWR06" H 2060 6235 50  0001 C CNN
 F 1 "GND" H 2065 6312 50  0000 C CNN
 F 2 "" H 2060 6485 50  0001 C CNN
@@
 $EndComp
 $Comp
-L GND #PWR3
+L GND #PWR07
 U 1 1 5B04308A
 P 1785 6485
-F 0 "#PWR3" H 1785 6235 50  0001 C CNN
+F 0 "#PWR07" H 1785 6235 50  0001 C CNN
 F 1 "GND" H 1790 6312 50  0000 C CNN
 F 2 "" H 1785 6485 50  0001 C CNN
@@
 $EndComp
 $Comp
-L GND #PWR7
+L GND #PWR08
 U 1 1 5B043F5D
 P 2705 7280
-F 0 "#PWR7" H 2705 7030 50  0001 C CNN
+F 0 "#PWR08" H 2705 7030 50  0001 C CNN
 F 1 "GND" H 2710 7107 50  0000 C CNN
 F 2 "" H 2705 7280 50  0001 C CNN
@@
 $EndComp
 $Comp
-L GND #PWR12
+L GND #PWR09
 U 1 1 5B044D4C
 P 4485 7315
-F 0 "#PWR12" H 4485 7065 50  0001 C CNN
+F 0 "#PWR09" H 4485 7065 50  0001 C CNN
 F 1 "GND" H 4490 7142 50  0000 C CNN
 F 2 "" H 4485 7315 50  0001 C CNN
@@
 $EndComp
 $Comp
-L GND #PWR22
+L GND #PWR010
 U 1 1 5B06F6EF
 P 9930 3790
-F 0 "#PWR22" H 9930 3540 50  0001 C CNN
+F 0 "#PWR010" H 9930 3540 50  0001 C CNN
 F 1 "GND" H 9935 3617 50  0000 C CNN
 F 2 "" H 9930 3790 50  0001 C CNN
@@
 $EndComp
 $Comp
-L GND #PWR20
+L GND #PWR011
 U 1 1 5B0753BB
 P 6760 3380
-F 0 "#PWR20" H 6760 3130 50  0001 C CNN
+F 0 "#PWR011" H 6760 3130 50  0001 C CNN
 F 1 "GND" H 6765 3207 50  0000 C CNN
 F 2 "" H 6760 3380 50  0001 C CNN
@@
 NoConn ~ 1465 4560
 $Comp
-L GND #PWR1
+L GND #PWR012
 U 1 1 5B081C3A
 P 1545 4710
-F 0 "#PWR1" H 1545 4460 50  0001 C CNN
+F 0 "#PWR012" H 1545 4460 50  0001 C CNN
 F 1 "GND" H 1550 4537 50  0000 C CNN
 F 2 "" H 1545 4710 50  0001 C CNN
@@
 $EndComp
 $Comp
-L GND #PWR18
+L GND #PWR013
 U 1 1 5B082DC4
 P 5880 3240
-F 0 "#PWR18" H 5880 2990 50  0001 C CNN
+F 0 "#PWR013" H 5880 2990 50  0001 C CNN
 F 1 "GND" H 5885 3067 50  0000 C CNN
 F 2 "" H 5880 3240 50  0001 C CNN
@@
 Connection ~ 10575 2935
 $Comp
-L GND #PWR23
+L GND #PWR014
 U 1 1 5B098D9A
 P 11070 2830
-F 0 "#PWR23" H 11070 2580 50  0001 C CNN
+F 0 "#PWR014" H 11070 2580 50  0001 C CNN
 F 1 "GND" H 11075 2657 50  0000 C CNN
 F 2 "" H 11070 2830 50  0001 C CNN
@@
 F 0 "CN3" H 3835 1100 50  0000 C CNN
 F 1 "SX1238_TRX_HEADER" H 3895 2224 50  0000 C CNN
-F 2 "Socket_Strips:Socket_Strip_Straight_2x10" H 3895 450 50  0001 C CNN
+F 2 "socket-strip-straight-2x10:sx1238_trx" H 3895 450 50  0001 C CNN
 F 3 "" H 3895 450 50  0001 C CNN
 	1    3895 1650
@@
 	2225 1540 2225 1670
 $Comp
-L GND #PWR5
+L GND #PWR015
 U 1 1 5B0A5E1E
 P 2225 1670
-F 0 "#PWR5" H 2225 1420 50  0001 C CNN
+F 0 "#PWR015" H 2225 1420 50  0001 C CNN
 F 1 "GND" H 2230 1497 50  0000 C CNN
 F 2 "" H 2225 1670 50  0001 C CNN
@@
 +3V3
 $Comp
-L GND #PWR8
+L GND #PWR016
 U 1 1 5B0AC996
 P 3070 1200
-F 0 "#PWR8" H 3070 950 50  0001 C CNN
+F 0 "#PWR016" H 3070 950 50  0001 C CNN
 F 1 "GND" H 3075 1027 50  0000 C CNN
 F 2 "" H 3070 1200 50  0001 C CNN
@@
 SPI2_SCK
 $Comp
-L GND #PWR9
+L GND #PWR017
 U 1 1 5B0AE690
 P 3070 1500
-F 0 "#PWR9" H 3070 1250 50  0001 C CNN
+F 0 "#PWR017" H 3070 1250 50  0001 C CNN
 F 1 "GND" H 3075 1327 50  0000 C CNN
 F 2 "" H 3070 1500 50  0001 C CNN
@@
 	4145 2100 4720 2100
 $Comp
-L GND #PWR13
+L GND #PWR018
 U 1 1 5B0AEB87
 P 4720 2100
-F 0 "#PWR13" H 4720 1850 50  0001 C CNN
+F 0 "#PWR018" H 4720 1850 50  0001 C CNN
 F 1 "GND" H 4725 1927 50  0000 C CNN
 F 2 "" H 4720 2100 50  0001 C CNN
@@
 	1625 3160 1695 3160
 $Comp
-L GND #PWR2
+L GND #PWR019
 U 1 1 5B0B10C1
 P 1695 3160
-F 0 "#PWR2" H 1695 2910 50  0001 C CNN
+F 0 "#PWR019" H 1695 2910 50  0001 C CNN
 F 1 "GND" H 1700 2987 50  0000 C CNN
 F 2 "" H 1695 3160 50  0001 C CNN
@@
 NRST
 $Comp
-L GND #PWR11
+L GND #PWR020
 U 1 1 5B0B8F14
 P 4200 3080
-F 0 "#PWR11" H 4200 2830 50  0001 C CNN
+F 0 "#PWR020" H 4200 2830 50  0001 C CNN
 F 1 "GND" H 4205 2907 50  0000 C CNN
 F 2 "" H 4200 3080 50  0001 C CNN
@@
 $EndComp
 $Comp
-L GND #PWR21
+L GND #PWR021
 U 1 1 5B0C38AE
 P 8160 5860
-F 0 "#PWR21" H 8160 5610 50  0001 C CNN
+F 0 "#PWR021" H 8160 5610 50  0001 C CNN
 F 1 "GND" H 8165 5687 50  0000 C CNN
 F 2 "" H 8160 5860 50  0001 C CNN
@@
 Connection ~ 6235 2750
 $Comp
-L GND #PWR19
+L GND #PWR022
 U 1 1 5B1AE42D
 P 6235 2785
-F 0 "#PWR19" H 6235 2535 50  0001 C CNN
+F 0 "#PWR022" H 6235 2535 50  0001 C CNN
 F 1 "GND" H 6315 2770 50  0000 C CNN
 F 2 "" H 6235 2785 50  0001 C CNN
@@
 	4855 4565 4855 5170
 $Comp
-L GND #PWR14
+L GND #PWR023
 U 1 1 5B1D46F6
 P 4855 5170
-F 0 "#PWR14" H 4855 4920 50  0001 C CNN
+F 0 "#PWR023" H 4855 4920 50  0001 C CNN
 F 1 "GND" H 4860 4997 50  0000 C CNN
 F 2 "" H 4855 5170 50  0001 C CNN

Commit message: more layout
Parts:
- added R15: 10K, Resistors_SMD:R_0603, symbol R_Small
- R4: value 0 -> 10K
Connections:
- net +VIN: now also R15.2; no longer U1.11 (EN)
- new net: R15.1, U1.11 (EN)
Changed lines of the file:
@@
 $EndComp
 $Comp
-L GND #PWR01
+L GND #PWR10
 U 1 1 5B041A53
 P 3720 7315
-F 0 "#PWR01" H 3720 7065 50  0001 C CNN
+F 0 "#PWR10" H 3720 7065 50  0001 C CNN
 F 1 "GND" H 3725 7142 50  0000 C CNN
 F 2 "" H 3720 7315 50  0001 C CNN
@@
 $EndComp
 $Comp
-L GND #PWR02
+L GND #PWR15
 U 1 1 5B041F18
 P 4975 6485
-F 0 "#PWR02" H 4975 6235 50  0001 C CNN
+F 0 "#PWR15" H 4975 6235 50  0001 C CNN
 F 1 "GND" H 4980 6312 50  0000 C CNN
 F 2 "" H 4975 6485 50  0001 C CNN
@@
 $EndComp
 $Comp
-L GND #PWR03
+L GND #PWR16
 U 1 1 5B04234F
 P 5255 6485
-F 0 "#PWR03" H 5255 6235 50  0001 C CNN
+F 0 "#PWR16" H 5255 6235 50  0001 C CNN
 F 1 "GND" H 5260 6312 50  0000 C CNN
 F 2 "" H 5255 6485 50  0001 C CNN
@@
 $EndComp
 $Comp
-L GND #PWR04
+L GND #PWR17
 U 1 1 5B0423C8
 P 5530 6485
-F 0 "#PWR04" H 5530 6235 50  0001 C CNN
+F 0 "#PWR17" H 5530 6235 50  0001 C CNN
 F 1 "GND" H 5535 6312 50  0000 C CNN
 F 2 "" H 5530 6485 50  0001 C CNN
@@
 $EndComp
 $Comp
-L GND #PWR05
+L GND #PWR6
 U 1 1 5B04306E
 P 2340 6485
-F 0 "#PWR05" H 2340 6235 50  0001 C CNN
+F 0 "#PWR6" H 2340 6235 50  0001 C CNN
 F 1 "GND" H 2345 6312 50  0000 C CNN
 F 2 "" H 2340 6485 50  0001 C CNN
@@
 $EndComp
 $Comp
-L GND #PWR06
+L GND #PWR4
 U 1 1 5B04307C
 P 2060 6485
-F 0 "#PWR06" H 2060 6235 50  0001 C CNN
+F 0 "#PWR4" H 2060 6235 50  0001 C CNN
 F 1 "GND" H 2065 6312 50  0000 C CNN
 F 2 "" H 2060 6485 50  0001 C CNN
@@
 $EndComp
 $Comp
-L GND #PWR07
+L GND #PWR3
 U 1 1 5B04308A
 P 1785 6485
-F 0 "#PWR07" H 1785 6235 50  0001 C CNN
+F 0 "#PWR3" H 1785 6235 50  0001 C CNN
 F 1 "GND" H 1790 6312 50  0000 C CNN
 F 2 "" H 1785 6485 50  0001 C CNN
@@
 $EndComp
 $Comp
-L GND #PWR08
+L GND #PWR7
 U 1 1 5B043F5D
 P 2705 7280
-F 0 "#PWR08" H 2705 7030 50  0001 C CNN
+F 0 "#PWR7" H 2705 7030 50  0001 C CNN
 F 1 "GND" H 2710 7107 50  0000 C CNN
 F 2 "" H 2705 7280 50  0001 C CNN
@@
 $EndComp
 $Comp
-L GND #PWR09
+L GND #PWR12
 U 1 1 5B044D4C
 P 4485 7315
-F 0 "#PWR09" H 4485 7065 50  0001 C CNN
+F 0 "#PWR12" H 4485 7065 50  0001 C CNN
 F 1 "GND" H 4490 7142 50  0000 C CNN
 F 2 "" H 4485 7315 50  0001 C CNN
@@
 Text Label 5780 6150 2    60   ~ 0
 +3V3
-Text Label 2600 6750 0    60   ~ 0
+Text Label 2315 6750 0    60   ~ 0
 +VIN
 $Comp
@@
 $EndComp
 $Comp
-L GND #PWR010
+L GND #PWR22
 U 1 1 5B06F6EF
 P 9930 3790
-F 0 "#PWR010" H 9930 3540 50  0001 C CNN
+F 0 "#PWR22" H 9930 3540 50  0001 C CNN
 F 1 "GND" H 9935 3617 50  0000 C CNN
 F 2 "" H 9930 3790 50  0001 C CNN
@@
 $EndComp
 $Comp
-L GND #PWR011
+L GND #PWR20
 U 1 1 5B0753BB
 P 6760 3380
-F 0 "#PWR011" H 6760 3130 50  0001 C CNN
+F 0 "#PWR20" H 6760 3130 50  0001 C CNN
 F 1 "GND" H 6765 3207 50  0000 C CNN
 F 2 "" H 6760 3380 50  0001 C CNN
@@
 NoConn ~ 1465 4560
 $Comp
-L GND #PWR012
+L GND #PWR1
 U 1 1 5B081C3A
 P 1545 4710
-F 0 "#PWR012" H 1545 4460 50  0001 C CNN
+F 0 "#PWR1" H 1545 4460 50  0001 C CNN
 F 1 "GND" H 1550 4537 50  0000 C CNN
 F 2 "" H 1545 4710 50  0001 C CNN
@@
 $EndComp
 $Comp
-L GND #PWR013
+L GND #PWR18
 U 1 1 5B082DC4
 P 5880 3240
-F 0 "#PWR013" H 5880 2990 50  0001 C CNN
+F 0 "#PWR18" H 5880 2990 50  0001 C CNN
 F 1 "GND" H 5885 3067 50  0000 C CNN
 F 2 "" H 5880 3240 50  0001 C CNN
@@
 	2505 6900 2820 6900
 Wire Wire Line
-	2820 6750 2600 6750
+	2535 6750 2315 6750
 Connection ~ 2060 6150
 Connection ~ 2340 6150
@@
 Connection ~ 10575 2935
 $Comp
-L GND #PWR014
+L GND #PWR23
 U 1 1 5B098D9A
 P 11070 2830
-F 0 "#PWR014" H 11070 2580 50  0001 C CNN
+F 0 "#PWR23" H 11070 2580 50  0001 C CNN
 F 1 "GND" H 11075 2657 50  0000 C CNN
 F 2 "" H 11070 2830 50  0001 C CNN
@@
 	2225 1540 2225 1670
 $Comp
-L GND #PWR015
+L GND #PWR5
 U 1 1 5B0A5E1E
 P 2225 1670
-F 0 "#PWR015" H 2225 1420 50  0001 C CNN
+F 0 "#PWR5" H 2225 1420 50  0001 C CNN
 F 1 "GND" H 2230 1497 50  0000 C CNN
 F 2 "" H 2225 1670 50  0001 C CNN
@@
 +3V3
 $Comp
-L GND #PWR016
+L GND #PWR8
 U 1 1 5B0AC996
 P 3070 1200
-F 0 "#PWR016" H 3070 950 50  0001 C CNN
+F 0 "#PWR8" H 3070 950 50  0001 C CNN
 F 1 "GND" H 3075 1027 50  0000 C CNN
 F 2 "" H 3070 1200 50  0001 C CNN
@@
 SPI2_SCK
 $Comp
-L GND #PWR017
+L GND #PWR9
 U 1 1 5B0AE690
 P 3070 1500
-F 0 "#PWR017" H 3070 1250 50  0001 C CNN
+F 0 "#PWR9" H 3070 1250 50  0001 C CNN
 F 1 "GND" H 3075 1327 50  0000 C CNN
 F 2 "" H 3070 1500 50  0001 C CNN
@@
 	4145 2100 4720 2100
 $Comp
-L GND #PWR018
+L GND #PWR13
 U 1 1 5B0AEB87
 P 4720 2100
-F 0 "#PWR018" H 4720 1850 50  0001 C CNN
+F 0 "#PWR13" H 4720 1850 50  0001 C CNN
 F 1 "GND" H 4725 1927 50  0000 C CNN
 F 2 "" H 4720 2100 50  0001 C CNN
@@
 	1625 3160 1695 3160
 $Comp
-L GND #PWR019
+L GND #PWR2
 U 1 1 5B0B10C1
 P 1695 3160
-F 0 "#PWR019" H 1695 2910 50  0001 C CNN
+F 0 "#PWR2" H 1695 2910 50  0001 C CNN
 F 1 "GND" H 1700 2987 50  0000 C CNN
 F 2 "" H 1695 3160 50  0001 C CNN
@@
 NRST
 $Comp
-L GND #PWR020
+L GND #PWR11
 U 1 1 5B0B8F14
 P 4200 3080
-F 0 "#PWR020" H 4200 2830 50  0001 C CNN
+F 0 "#PWR11" H 4200 2830 50  0001 C CNN
 F 1 "GND" H 4205 2907 50  0000 C CNN
 F 2 "" H 4200 3080 50  0001 C CNN
@@
 $EndComp
 $Comp
-L GND #PWR021
+L GND #PWR21
 U 1 1 5B0C38AE
 P 8160 5860
-F 0 "#PWR021" H 8160 5610 50  0001 C CNN
+F 0 "#PWR21" H 8160 5610 50  0001 C CNN
 F 1 "GND" H 8165 5687 50  0000 C CNN
 F 2 "" H 8160 5860 50  0001 C CNN
@@
 P 2505 7090
 F 0 "R4" H 2545 7125 50  0000 L CNN
-F 1 "0" V 2505 7065 50  0000 L CNN
+F 1 "10K" V 2505 7015 50  0000 L CNN
 F 2 "Resistors_SMD:R_0603" H 2505 7090 50  0001 C CNN
 F 3 "" H 2505 7090 50  0001 C CNN
@@
 Connection ~ 6235 2750
 $Comp
-L GND #PWR022
+L GND #PWR19
 U 1 1 5B1AE42D
 P 6235 2785
-F 0 "#PWR022" H 6235 2535 50  0001 C CNN
+F 0 "#PWR19" H 6235 2535 50  0001 C CNN
 F 1 "GND" H 6315 2770 50  0000 C CNN
 F 2 "" H 6235 2785 50  0001 C CNN
@@
 	4855 4565 4855 5170
 $Comp
-L GND #PWR023
+L GND #PWR14
 U 1 1 5B1D46F6
 P 4855 5170
-F 0 "#PWR023" H 4855 4920 50  0001 C CNN
+F 0 "#PWR14" H 4855 4920 50  0001 C CNN
 F 1 "GND" H 4860 4997 50  0000 C CNN
 F 2 "" H 4855 5170 50  0001 C CNN
@@
 	10395 2735 10770 2735
 Connection ~ 10575 2735
+$Comp
+L R_Small R15
+U 1 1 5B21B026
+P 2635 6750
+F 0 "R15" V 2570 6750 50  0000 C CNN
+F 1 "10K" V 2635 6750 50  0000 C CNN
+F 2 "Resistors_SMD:R_0603" H 2635 6750 50  0001 C CNN
+F 3 "" H 2635 6750 50  0001 C CNN
+	1    2635 6750
+	0    1    1    0
+$EndComp
+Wire Wire Line
+	2735 6750 2820 6750
 $EndSCHEMATC
